File: board/hw/control.brd (EAGLE design)
At the start: 54.3 x 82.5 mm, 34 parts, among them T1 pn2222a, T2 pn2222a, T3 pn2222a, T4 pn2222a, T5 pn2222a, T6 pn2222a, T7 pn2222a, T8 pn2222a

Commit message: moved everything to a bottom layer
Parts:
- flipped C2 to the bottom, turned to 0 degrees
- flipped C3 to the bottom
- flipped C4 to the bottom
- flipped R1 to the bottom, turned to 0 degrees
- flipped R2 to the bottom, turned to 0 degrees
- flipped R3 to the bottom, turned to 0 degrees
- flipped R4 to the bottom, turned to 180 degrees
- flipped R5 to the bottom, turned to 180 degrees
- flipped R6 to the bottom, turned to 180 degrees
- flipped R7 to the bottom, turned to 180 degrees
- flipped R8 to the bottom, turned to 0 degrees
- flipped R9 to the bottom, turned to 0 degrees
Routing:
- added copper zone on layer 16, net 0V
- removed copper zone on layer 1, net 0V
Other:
- board text added: "Lemur's Bobik v1.0"
